Commit message: Added CAD and modified some parameters

File: src/modelrocket.urdf (robot description, URDF)
Before this commit: robot rocket, 7 links, 6 joints
Links:
- removed link booster_link
- removed link leg_1
- removed link leg_2
- removed link leg_3
- removed link top_hat_link
- removed link top_link
- link base_link: mass 91.0 -> 91; geometry collision mesh filename=/Users/alexpinel/Desktop/PyRocketCraft/Instinct V2 v3.stl scale=2 2 2; visual mesh filename=/Users/alexpinel/Desktop/PyRocketCraft/Instinct V2 v3.stl scale=2 2 2
Joints:
- removed joint booster_joint
- removed joint leg_1_joint
- removed joint leg_2_joint
- removed joint leg_3_joint
- removed joint top_hat_joint
- removed joint top_joint
